Commit message: docker desktop reboot commit

File: src/simulator/model/main_car/urdf/main_car.urdf (robot description, URDF)
Before this commit: robot main_car, 7 links, 6 joints
Links:
- link back_right_wheel_rot: mass 0.0632357163080608 -> 0.0632357163080607
- link base_link: mass 0.58722731346914 -> 0.616866978201299
Joints:
- joint back_right_wheel_rot_j: origin xyz=0.166149999999796 0.00849999999999998 0.0147 rpy=0 0 0 -> xyz=0.16615 0.0085 0.0147 rpy=0 0 0
- joint front_left_wheel_steer_j: origin xyz=-0.0212429479041969 0.211254558119221 0.0117 rpy=0 0 0 -> xyz=-0.021243 0.21125 0.0117 rpy=0 0 0
- joint front_right_wheel_rot_j: axis 0.999773526729787 -0.0212813357260373 0 -> 0.99977 -0.021281 0; origin xyz=0.131001462865903 0.210751140085241 0.0117 rpy=0 0 0 -> xyz=0.131 0.21075 0.0117 rpy=0 0 0
- joint front_right_wheel_steer_j: origin xyz=0.131001462865903 0.210751140085241 0.0117 rpy=0 0 0 -> xyz=0.131 0.21075 0.0117 rpy=0 0 0
